Commit message: Exp2 NMPCC suite: slender/grasp_pose scenes, diagnostics extraction, y_guard removal; drop legacy v1 files

File: openarmx_ros2_visual_mujoco.urdf (robot description, URDF)
Before this commit: robot openarmx, 30 links, 29 joints
Links:
- removed link openarmx_left_left_finger
- removed link openarmx_left_right_finger
- removed link openarmx_right_left_finger
- removed link openarmx_right_right_finger
- link openarmx_body_link0: geometry collision mesh filename=D:\RobotSim\openarmx_mujoco\ros2_visual_meshes\body\v10\vis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 scale=1.0 1.0 1.0; visual mesh filename=D:\RobotSim\openarmx_mujoco\ros2_visual_meshes\body\v10\vis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 scale=1.0 1.0 1.0
- link openarmx_left_hand: geometry collision mesh filename=D:\RobotSim\openarmx_mujoco\ros2_visual_meshes\ee\openarmx_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 scale=0.001 0.001 0.001; collision mesh filename=D:\RobotSim\openarmx_mujoco\ros2_visual_meshes\ee\openarmx_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 scale=0.001 0.001 0.001
- link openarmx_left_link0: geometry collision mesh filename=D:\RobotSim\openarmx_mujoco\ros2_visual_meshes\arm\v10\visu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 scale=1.0 1.0 1.0; collision mesh filename=D:\RobotSim\openarmx_mujoco\ros2_visual_meshes\arm\v10\visu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 scale=1.0 1.0 1.0
- link openarmx_left_link1: geometry collision mesh filename=D:\RobotSim\openarmx_mujoco\ros2_visual_meshes\arm\v10\visu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 scale=1.0 1.0 1.0; collision mesh filename=D:\RobotSim\openarmx_mujoco\ros2_visual_meshes\arm\v10\visu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 scale=1.0 1.0 1.0
- link openarmx_left_link2: geometry collision mesh filename=D:\RobotSim\openarmx_mujoco\ros2_visual_meshes\arm\v10\visu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 scale=1.0 1.0 1.0; collision mesh filename=D:\RobotSim\openarmx_mujoco\ros2_visual_meshes\arm\v10\visu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 scale=1.0 1.0 1.0
- link openarmx_left_link3: geometry collision mesh filename=D:\RobotSim\openarmx_mujoco\ros2_visual_meshes\arm\v10\visu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 scale=1.0 1.0 1.0; collision mesh filename=D:\RobotSim\openarmx_mujoco\ros2_visual_meshes\arm\v10\visu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 scale=1.0 1.0 1.0
- link openarmx_left_link4: geometry collision mesh filename=D:\RobotSim\openarmx_mujoco\ros2_visual_meshes\arm\v10\visu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 scale=1.0 1.0 1.0; collision mesh filename=D:\RobotSim\openarmx_mujoco\ros2_visual_meshes\arm\v10\visu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 scale=1.0 1.0 1.0
- link openarmx_left_link5: geometry collision mesh filename=D:\RobotSim\openarmx_mujoco\ros2_visual_meshes\arm\v10\visu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 scale=1.0 1.0 1.0; collision mesh filename=D:\RobotSim\openarmx_mujoco\ros2_visual_meshes\arm\v10\visu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 scale=1.0 1.0 1.0
- link openarmx_left_link6: geometry collision mesh filename=D:\RobotSim\openarmx_mujoco\ros2_visual_meshes\arm\v10\visu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 scale=1.0 1.0 1.0; collision mesh filename=D:\RobotSim\openarmx_mujoco\ros2_visual_meshes\arm\v10\visu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 scale=1.0 1.0 1.0
- link openarmx_left_link7: geometry collision mesh filename=D:\RobotSim\openarmx_mujoco\ros2_visual_meshes\arm\v10\visu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 scale=1.0 1.0 1.0; collision mesh filename=D:\RobotSim\openarmx_mujoco\ros2_visual_meshes\arm\v10\visu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 scale=1.0 1.0 1.0
- link openarmx_right_hand: geometry collision mesh filename=D:\RobotSim\openarmx_mujoco\ros2_visual_meshes\ee\openarmx_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 scale=0.001 0.001 0.001; collision mesh filename=D:\RobotSim\openarmx_mujoco\ros2_visual_meshes\ee\openarmx_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 scale=0.001 0.001 0.001
- link openarmx_right_link0: geometry collision mesh filename=D:\RobotSim\openarmx_mujoco\ros2_visual_meshes\arm\v10\visu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 scale=1.0 1.0 1.0; collision mesh filename=D:\RobotSim\openarmx_mujoco\ros2_visual_meshes\arm\v10\visu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 scale=1.0 1.0 1.0
- link openarmx_right_link1: geometry collision mesh filename=D:\RobotSim\openarmx_mujoco\ros2_visual_meshes\arm\v10\visu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 scale=1.0 1.0 1.0; collision mesh filename=D:\RobotSim\openarmx_mujoco\ros2_visual_meshes\arm\v10\visu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 scale=1.0 1.0 1.0
- link openarmx_right_link2: geometry collision mesh filename=D:\RobotSim\openarmx_mujoco\ros2_visual_meshes\arm\v10\visu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 scale=1.0 1.0 1.0; collision mesh filename=D:\RobotSim\openarmx_mujoco\ros2_visual_meshes\arm\v10\visu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 scale=1.0 1.0 1.0
- link openarmx_right_link3: geometry collision mesh filename=D:\RobotSim\openarmx_mujoco\ros2_visual_meshes\arm\v10\visu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 scale=1.0 1.0 1.0; collision mesh filename=D:\RobotSim\openarmx_mujoco\ros2_visual_meshes\arm\v10\visu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 scale=1.0 1.0 1.0
- link openarmx_right_link4: geometry collision mesh filename=D:\RobotSim\openarmx_mujoco\ros2_visual_meshes\arm\v10\visu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 scale=1.0 1.0 1.0; collision mesh filename=D:\RobotSim\openarmx_mujoco\ros2_visual_meshes\arm\v10\visu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 scale=1.0 1.0 1.0
- link openarmx_right_link5: geometry collision mesh filename=D:\RobotSim\openarmx_mujoco\ros2_visual_meshes\arm\v10\visu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 scale=1.0 1.0 1.0; collision mesh filename=D:\RobotSim\openarmx_mujoco\ros2_visual_meshes\arm\v10\visu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 scale=1.0 1.0 1.0
- link openarmx_right_link6: geometry collision mesh filename=D:\RobotSim\openarmx_mujoco\ros2_visual_meshes\arm\v10\visu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 scale=1.0 1.0 1.0; collision mesh filename=D:\RobotSim\openarmx_mujoco\ros2_visual_meshes\arm\v10\visu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 scale=1.0 1.0 1.0
- link openarmx_right_link7: geometry collision mesh filename=D:\RobotSim\openarmx_mujoco\ros2_visual_meshes\arm\v10\visu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 scale=1.0 1.0 1.0; collision mesh filename=D:\RobotSim\openarmx_mujoco\ros2_visual_meshes\arm\v10\visu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 scale=1.0 1.0 1.0
Joints:
- removed joint openarmx_left_finger_joint1
- removed joint openarmx_left_finger_joint2
- removed joint openarmx_right_finger_joint1
- removed joint openarmx_right_finger_joint2
